Commit message: Add files via upload

File: BRT_Description/urdf/BRT_Gazebo.urdf (robot description, URDF)
Before this commit: robot braccio, 9 links, 8 joints
Links:
- link braccio_base_link: mass 0.1 -> 0.16
- link elbow_link: mass 0.1 -> 0.169
- link left_gripper_link: mass 0.1 -> 0.002; geometry collision mesh filename=package://BRT_Description/stl/braccio_left_gripper.stl scale=0.001 0.001 0.001; visual mesh filename=package://BRT_Description/stl/braccio_left_gripper.stl scale=0.001 0.001 0.001
- link right_gripper_link: mass 0.1 -> 0.002; geometry collision mesh filename=package://BRT_Description/stl/braccio_right_gripper.stl scale=0.001 0.001 0.001; visual mesh filename=package://BRT_Description/stl/braccio_right_gripper.stl scale=0.001 0.001 0.001
- link shoulder_link: mass 0.1 -> 0.16
- link wrist_pitch_link: mass 0.1 -> 0.062
- link wrist_roll_link: mass 0.1 -> 0.022

Commit message: Add files via upload

File: BRT_Description/urdf/BRT_Gazebo.urdf (robot description, URDF)
Before this commit: robot braccio, 9 links, 8 joints
Links:
- added link camera_link, mass 1e-5; collision box size=0.03 0.06 0.03; visual box size=0.03 0.06 0.03
- added link camera_rgb_frame
- added link camera_rgb_optical_frame
Joints:
- added joint camera_rgb_joint: type fixed, parent camera_link, child camera_rgb_frame, origin xyz=0.003 0.011 0.009 rpy=0 0 0
- added joint camera_rgb_optical_joint: type fixed, parent camera_rgb_frame, child camera_rgb_optical_frame, origin xyz=0 0 0 rpy=-1.57 0 -1.57
- added joint table_joint: type fixed, parent world, child camera_link, origin xyz=0.0 0.7 0.15 rpy=0 0 -1.57
