Commit message: Add files via upload

File: BRT_Description/urdf/BRT.urdf (robot description, URDF)
Before this commit: robot Braccio, 9 links, 8 joints
Links:
- link left_gripper_link: geometry visual mesh filename=package://BRT_Description/meshes/braccio_left_gripper.stl scale=0.01 0.01 0.01
- link right_gripper_link: geometry visual mesh filename=package://BRT_Description/meshes/braccio_right_gripper.stl scale=0.01 0.01 0.01

File: BRT_Description/urdf/BRT_Gazebo.urdf (robot description, URDF)
Before this commit: robot braccio, 12 links, 11 joints
Links:
- link left_gripper_link: geometry collision mesh filename=package://BRT_Description/meshes/braccio_left_gripper.stl scale=0.01 0.01 0.01; visual mesh filename=package://BRT_Description/meshes/braccio_left_gripper.stl scale=0.01 0.01 0.01
- link right_gripper_link: geometry collision mesh filename=package://BRT_Description/meshes/braccio_right_gripper.stl scale=0.01 0.01 0.01; visual mesh filename=package://BRT_Description/meshes/braccio_right_gripper.stl scale=0.01 0.01 0.01
Joints:
- joint table_joint: origin xyz=0.0 0.7 0.15 rpy=0 0 -1.57 -> xyz=0.0 0.45 0.3 rpy=0 0 -1.57

File: BRT_Description/urdf/BRT_model.urdf (robot description, URDF)
Before this commit: robot BRT, 9 links, 8 joints
Links:
- link left_gripper_link: geometry collision mesh filename=package://BRT_Description/meshes/braccio_left_gripper.stl scale=0.01 0.01 0.01; visual mesh filename=package://BRT_Description/meshes/braccio_left_gripper.stl scale=0.01 0.01 0.01
- link right_gripper_link: geometry collision mesh filename=package://BRT_Description/meshes/braccio_right_gripper.stl scale=0.01 0.01 0.01; visual mesh filename=package://BRT_Description/meshes/braccio_right_gripper.stl scale=0.01 0.01 0.01
